File: BudgetJoycons_pcb/BudgetJoycons_pcb.kicad_pcb (KiCad board)
At the start: 4 copper layers, 39.1 x 94.5 mm, 111 parts, among them J1 S2B-PH-K-SLFSN, J2 UJ20-C-H-G-SMT-2A-P16-TR, J3 530480210, J4 PCB Pads, Q1 AO3401A, Q2 AO3401A, Q3 AO3400A, Q4 AO3401A, Q5 AO3401A, Q6 AO3400A, SW1 B3F_1020, SW10 SKSCLBE010, SW11 SKSCLBE010, SW12 SKSCLBE010, SW2 TL3315NF100Q, SW3 TL3315NF100Q, SW4 TL3315NF100Q, SW5 TL3315NF100Q, SW6 TL3315NF100Q, SW7 TL3315NF100Q, SW8 TL3315NF100Q, SW9 SKSCLBE010, U1 STM32C071CBT6, U2 NRF24L01_Breakout, U3 AP2127K-3.3, U4 MCP73831-2-OT, U5 USBLC6-2SC6, U6 DRV5056A3, U7 DRV5056A3, U8 DRV5056A3, U9 LSM6DSM

Commit message: Right PCB update
Parts:
- removed H1, H2, H3, H4: MountingHole_Pad, MountingHole:MountingHole_3mm_Pad
- removed H5, H6: MountingHole, MountingHole:MountingHole_3mm
- C1, C14, C15, C16, C17, C18, C19, C2, C20, C21, C22, C3, C6, C7, D9, Q4, Q5, Q6, R28, R29, R3, R32, R33, R34, R38, R39, R40, R5, SW9, U5, U6, U7, U8: moved to B.Cu
- moved C2 132.4 mm to (152.3, 76.8), turned to 45 degrees
- moved C24 120.5 mm to (145.5, 71.6), turned to 180 degrees
- moved C6 118.2 mm to (143.8, 141.2), turned to 90 degrees
- moved U9 116.1 mm to (141.7, 71.1), turned to 90 degrees
- moved D1 113.7 mm to (158.4, 92.3), turned to -90 degrees
- moved D2 113.6 mm to (158.4, 96.1), turned to -90 degrees
- moved D3 113.5 mm to (158.4, 99.9), turned to -90 degrees
- moved D4 113.3 mm to (158.4, 103.8), turned to -90 degrees
- moved R16 107.1 mm to (156.3, 92.3), turned to -90 degrees
- moved R4 107.1 mm to (154.2, 133.6), turned to -90 degrees
- moved R17 106.9 mm to (156.3, 96.1), turned to -90 degrees
- moved R18 106.8 mm to (156.3, 99.9), turned to -90 degrees
- moved R19 106.6 mm to (156.3, 103.8), turned to -90 degrees
- moved C7 106.1 mm to (145.7, 141.5), turned to 90 degrees
- moved R20 105.4 mm to (153.9, 140.8), turned to -90 degrees
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Connections:
- U5 pad 1: USB_D+ -> unconnected-(U5-I/O1-Pad1)
- U5 pad 3: USB_D- -> unconnected-(U5-I/O2-Pad3)
- U5 pad 4: unconnected-(U5-I/O3-Pad4) -> USB_D+
- U5 pad 6: unconnected-(U5-I/O4-Pad6) -> USB_D-
