File: BudgetJoycons_pcb/budgetJoycons_page2.kicad_sch (KiCad schematic)
At the start: 59 parts, among them J1 S2B-PH-K-SLFSN, J2 UJ20-C-H-G-SMT-2A-P16-TR, J3 530480210, Q1 AO3401A, Q2 AO3401A, Q3 AO3400A, Q4 AO3401A, Q5 AO3401A, Q6 AO3400A, SW10 SKSCLBE010, SW11 SKSCLBE010, SW12 SKSCLBE010, SW9 SKSCLBE010, U3 AP2127K-3.3, U4 MCP73831-2-OT, U5 USBLC6-2SC6, U6 DRV5056A3, U7 DRV5056A3, U8 DRV5056A3

Commit message: Right PCB update
Connections:
- net USB_D+: now also U5.4 (I/O3); no longer U5.1 (I/O1)
- net USB_D-: now also U5.6 (I/O4); no longer U5.3 (I/O2)
Changed lines of the file:
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@@
-	(wire
-		(pts
-			(xy 77.47 63.5) (xy 77.47 46.99)
-		)
-		(stroke
-			(width 0)
-			(type default)
-		)
-	)
 	(wire
 		(pts
@@
 	(wire
 		(pts
+			(xy 74.93 44.45) (xy 74.93 71.12)
+		)
+		(stroke
+			(width 0)
+			(type default)
+		)
+	)
+	(wire
+		(pts
 			(xy 237.49 85.09) (xy 241.3 85.09)
 		)
@@
 	(wire
 		(pts
-			(xy 80.01 66.04) (xy 74.93 66.04)
-		)
-		(stroke
-			(width 0)
-			(type default)
-		)
-	)
-	(wire
-		(pts
 			(xy 50.8 80.01) (xy 50.8 82.55)
 		)
@@
 	(wire
 		(pts
-			(xy 80.01 63.5) (xy 77.47 63.5)
-		)
-		(stroke
-			(width 0)
-			(type default)
-		)
-	)
-	(wire
-		(pts
 			(xy 246.38 74.93) (xy 246.38 77.47)
 		)
@@
 	(wire
 		(pts
+			(xy 77.47 46.99) (xy 77.47 68.58)
+		)
+		(stroke
+			(width 0)
+			(type default)
+		)
+	)
+	(wire
+		(pts
 			(xy 77.47 102.87) (xy 77.47 104.14)
 		)
@@
 	(wire
 		(pts
+			(xy 77.47 68.58) (xy 80.01 68.58)
+		)
+		(stroke
+			(width 0)
+			(type default)
+		)
+	)
+	(wire
+		(pts
 			(xy 201.93 35.56) (xy 201.93 36.83)
 		)
@@
 	(wire
 		(pts
-			(xy 74.93 66.04) (xy 74.93 44.45)
-		)
-		(stroke
-			(width 0)
-			(type default)
-		)
-	)
-	(wire
-		(pts
 			(xy 223.52 140.97) (xy 223.52 142.24)
 		)
@@
 		)
 		(stroke
+			(width 0)
+			(type default)
+		)
+	)
+	(wire
+		(pts
+			(xy 74.93 71.12) (xy 80.01 71.12)
+		)
+		(stroke
