File: BudgetJoycons_pcb/budgetJoycons_page3.kicad_sch (KiCad schematic)
At the start: 10 parts, among them J4 PCB Pads, U9 LSM6DSM

Commit message: Right PCB update
Parts:
- removed H1, H2, H3, H4: MountingHole_Pad, MountingHole:MountingHole_3mm_Pad, symbol Mechanical:MountingHole_Pad
- removed H5, H6: MountingHole, MountingHole:MountingHole_3mm, symbol Mechanical:MountingHole
Other:
- note removed: "MOUNTING"
